Commit message: full URDF without gripper

File: jdcobot200_urdf/jdcobot200.urdf (robot description, URDF)
Before this commit: robot jdcobot200_urdf, 2 links, 1 joints
Links:
- added link arm_link_assembly, mass 1e-09; collision mesh filename=ac1.stl; collision mesh filename=ac2.stl
- added link arm_link_assembly_2, mass 1e-09; collision mesh filename=ac1.stl; collision mesh filename=ac2.stl
- added link gripper_assembly, mass 1e-09; collision mesh filename=ac1.stl; collision mesh filename=ac2.stl
- added link wrist_assembly, mass 1e-09; collision mesh filename=ac1.stl; collision mesh filename=main.stl
Joints:
- added joint elbow: type revolute, parent arm_link_assembly, child arm_link_assembly_2, origin xyz=0.1352 8.02902e-05 -0.000107107 rpy=0 -0 -0, axis 0 0 1, limit lower=-3.141592653589793 upper=3.141592653589793 effort=10 velocity=10
- added joint gripper_base: type revolute, parent wrist_assembly, child gripper_assembly, origin xyz=0.0575 0 0.0183929 rpy=-3.14159 -1.5708 0, axis 0 0 1, limit lower=-3.141592653589793 upper=3.141592653589793 effort=10 velocity=10
- added joint shoulder: type revolute, parent shoulder_assmebly, child arm_link_assembly, origin xyz=-0.0184 0 -0.06146 rpy=-0 1.5708 0, axis 0 0 1, limit lower=-3.141592653589793 upper=3.141592653589793 effort=10 velocity=10
- added joint wrist: type revolute, parent arm_link_assembly_2, child wrist_assembly, origin xyz=0.1352 8.02902e-05 -0.000107107 rpy=0 0 -0, axis 0 0 1, limit lower=-3.141592653589793 upper=3.141592653589793 effort=10 velocity=10
