Commit message: June 22th

File: 2_jdcobot200_FK/1_URDF_visualize/jdcobot200.urdf (robot description, URDF)
Before this commit: robot jdcobot200_urdf, 8 links, 7 joints
Links:
- link arm_link_assembly: geometry collision mesh filename=ac1.stl; collision mesh filename=ac2.stl
- link arm_link_assembly_2: geometry collision mesh filename=ac1.stl; collision mesh filename=ac2.stl
- link base_assembly: geometry collision mesh filename=ac1.stl; collision mesh filename=base_link.stl
- link gripper_assembly: geometry collision mesh filename=ac1.stl; collision mesh filename=ac2.stl
- link gripper_left_assembly: geometry collision mesh filename=gripper_left.stl; visual mesh filename=gripper_left.stl
- link gripper_right_assembly: geometry collision mesh filename=gripper_right.stl; collision mesh filename=gripper_right_part.stl
- link shoulder_assmebly: geometry collision mesh filename=ac1.stl; collision mesh filename=ac2.stl
- link wrist_assembly: geometry collision mesh filename=ac1.stl; collision mesh filename=main.stl

File: 2_jdcobot200_FK/2_URDF_to_MJCF/jdcobot200.urdf (robot description, URDF)
Before this commit: robot jdcobot200_urdf, 8 links, 7 joints
Links:
- link arm_link_assembly: geometry collision mesh filename=ac1.stl; collision mesh filename=ac2.stl
- link arm_link_assembly_2: geometry collision mesh filename=ac1.stl; collision mesh filename=ac2.stl
- link base_assembly: geometry collision mesh filename=ac1.stl; collision mesh filename=base_link.stl
- link gripper_assembly: geometry collision mesh filename=ac1.stl; collision mesh filename=ac2.stl
- link gripper_left_assembly: geometry collision mesh filename=gripper_left.stl; visual mesh filename=gripper_left.stl
- link gripper_right_assembly: geometry collision mesh filename=gripper_right.stl; collision mesh filename=gripper_right_part.stl
- link shoulder_assmebly: geometry collision mesh filename=ac1.stl; collision mesh filename=ac2.stl
- link wrist_assembly: geometry collision mesh filename=ac1.stl; collision mesh filename=main.stl
